File: pcb/controller_mipi/t20_controller.kicad_sch (KiCad schematic)
At the start: 0 parts

Commit message: USB clean up
Other:
- removed sheet CV
- removed sheet FPGA_USB3
- removed sheet USB3
Changed lines of the file:
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@@
 (kicad_sch (version 20230819) (generator eeschema)
   (paper "A4")
-  (wire (pts (xy 224.79 128.27) (xy 234.95 128.27))
-    (stroke (width 0) (type default))
-  )
-  (wire (pts (xy 224.79 109.22) (xy 234.95 109.22))
-    (stroke (width 0) (type default))
-  )
-  (bus (pts (xy 224.79 101.6) (xy 234.95 101.6))
-    (stroke (width 0) (type default))
-  )
-  (wire (pts (xy 224.79 114.3) (xy 234.95 114.3))
-    (stroke (width 0) (type default))
-  )
-  (wire (pts (xy 224.79 125.73) (xy 234.95 125.73))
-    (stroke (width 0) (type default))
-  )
-  (wire (pts (xy 224.79 120.65) (xy 234.95 120.65))
-    (stroke (width 0) (type default))
-  )
-  (wire (pts (xy 224.79 106.68) (xy 234.95 106.68))
-    (stroke (width 0) (type default))
-  )
-  (wire (pts (xy 224.79 123.19) (xy 234.95 123.19))
-    (stroke (width 0) (type default))
-  )
-  (wire (pts (xy 224.79 111.76) (xy 234.95 111.76))
-    (stroke (width 0) (type default))
-  )
   (sheet (at 118.11 26.67) (size 36.83 33.02) (fields_autoplaced)
     (stroke (width 0.1524) (type solid) (color 26 255 5 1))
@@
     )
   )
-  (sheet (at 53.34 83.82) (size 40.64 26.67) (fields_autoplaced)
+  (sheet (at 31.75 69.85) (size 40.64 26.67) (fields_autoplaced)
     (stroke (width 0.1524) (type solid) (color 255 68 26 1))
     (fill (color 255 145 0 0.0800))
-    (property "Sheetname" "FPGA_PWR" (at 53.34 83.1084 0)
+    (property "Sheetname" "FPGA_PWR" (at 31.75 69.1384 0)
       (effects (font (size 1.27 1.27)) (justify left bottom))
     )
-    (property "Sheetfile" "FPGA_PWR.kicad_sch" (at 53.34 111.0746 0)
+    (property "Sheetfile" "FPGA_PWR.kicad_sch" (at 31.75 97.1046 0)
       (effects (font (size 1.27 1.27)) (justify left top))
     )
@@
       (project "t20_controller"
         (path "/ff96e853-bc79-4d79-a4a3-af9aaf1cbd33" (page "4"))
-      )
-    )
-  )
-  (sheet (at 234.95 88.9) (size 24.13 44.45) (fields_autoplaced)
-    (stroke (width 0.1524) (type solid))
-    (fill (color 255 0 105 0.0800))
-    (property "Sheetname" "USB3" (at 234.95 88.1884 0)
-      (effects (font (size 1.27 1.27)) (justify left bottom))
-    )
-    (property "Sheetfile" "USB3.kicad_sch" (at 234.95 133.9346 0)
-      (effects (font (size 1.27 1.27)) (justify left top))
-    )
-    (pin "HSPI_D[0..7]" bidirectional (at 234.95 101.6 180)
-      (effects (font (size 1.27 1.27)) (justify left))
-    )
-    (pin "HTRDY" input (at 234.95 111.76 180)
-      (effects (font (size 1.27 1.27)) (justify left))
-    )
-    (pin "HTCLK" output (at 234.95 106.68 180)
-      (effects (font (size 1.27 1.27)) (justify left))
-    )
-    (pin "HTREQ" output (at 234.95 109.22 180)
-      (effects (font (size 1.27 1.27)) (justify left))
-    )
-    (pin "HTACK" output (at 234.95 125.73 180)
-      (effects (font (size 1.27 1.27)) (justify left))
-    )
-    (pin "HTVLD" output (at 234.95 114.3 180)
-      (effects (font (size 1.27 1.27)) (justify left))
-    )
-    (pin "HRCLK" input (at 234.95 120.65 180)
-      (effects (font (size 1.27 1.27)) (justify left))
-    )
-    (pin "HRVLD" input (at 234.95 128.27 180)
-      (effects (font (size 1.27 1.27)) (justify left))
-    )
-    (pin "HRACT" input (at 234.95 123.19 180)
-      (effects (font (size 1.27 1.27)) (justify left))
-    )
-    (instances
-      (project "t20_controller"
-        (path "/ff96e853-bc79-4d79-a4a3-af9aaf1cbd33" (page "6"))
       )
     )
@@
     )
   )
-  (sheet (at 121.92 120.65) (size 48.26 35.56) (fields_autoplaced)
-    (stroke (width 0.1524) (type solid))
-    (fill (color 0 0 0 0.0000))
-    (property "Sheetname" "CV" (at 121.92 119.9384 0)
-      (effects (font (size 1.27 1.27)) (justify left bottom))
-    )
-    (property "Sheetfile" "CV.kicad_sch" (at 121.92 156.7946 0)
-      (effects (font (size 1.27 1.27)) (justify left top))
-    )
-    (instances
-      (project "t20_controller"
-        (path "/ff96e853-bc79-4d79-a4a3-af9aaf1cbd33" (page "8"))
-      )
-    )
-  )
   (sheet (at 163.83 29.21) (size 46.99 29.21) (fields_autoplaced)
     (stroke (width 0.1524) (type solid))
@@
       )
     )
-  )
-  (sheet (at 196.85 88.9) (size 27.94 44.45) (fields_autoplaced)
-    (stroke (width 0.1524) (type solid))
-    (fill (color 30 63 255 0.1200))
-    (property "Sheetname" "FPGA_USB3" (at 196.85 88.1884 0)
-      (effects (font (size 1.27 1.27)) (justify left bottom))
-    )
-    (property "Sheetfile" "FPGA_USB3.kicad_sch" (at 196.85 133.9346 0)
-      (effects (font (size 1.27 1.27)) (justify left top))
-    )
-    (pin "HSPI_D[0..7]" bidirectional (at 224.79 101.6 0)
-      (effects (font (size 1.27 1.27)) (justify right))
-    )
-    (pin "HTVLD" output (at 224.79 128.27 0)
-      (effects (font (size 1.27 1.27)) (justify right))
-    )
-    (pin "HRVLD" input (at 224.79 114.3 0)
-      (effects (font (size 1.27 1.27)) (justify right))
-    )
-    (pin "HTACK" output (at 224.79 111.76 0)
-      (effects (font (size 1.27 1.27)) (justify right))
-    )
-    (pin "HRACT" input (at 224.79 109.22 0)
-      (effects (font (size 1.27 1.27)) (justify right))
-    )
-    (pin "HRCLK" input (at 224.79 106.68 0)
-      (effects (font (size 1.27 1.27)) (justify right))
-    )
-    (pin "HTCLK" output (at 224.79 120.65 0)
-      (effects (font (size 1.27 1.27)) (justify right))
-    )
-    (pin "HTREQ" output (at 224.79 123.19 0)
-      (effects (font (size 1.27 1.27)) (justify right))
-    )
-    (pin "HTRDY" input (at 224.79 125.73 0)
-      (effects (font (size 1.27 1.27)) (justify right))
-    )
-    (instances
-      (project "t20_controller"
-        (path "/ff96e853-bc79-4d79-a4a3-af9aaf1cbd33" (page "7"))
-      )
-    )
